File: uterotrack.kicad_pcb (KiCad board)
At the start: 4 copper layers, 34 x 98 mm, 139 parts, among them J1 RFShield, J2 MicroSD_Card, J3 Argos_Prog, J4 AS5510, J5 Prog, J6 EXP, Q1 DMP2110UW, Q10 MMBT2222, Q11 MMBT2222, Q12 MMBT2222, Q13 MMBT2222, Q14 SiS454DN, Q15 SiS454DN, Q16 SiS415DNT, Q17 MMBT4403, Q18 MMBT2222, Q2 DMP2110UW, Q3 MMBT2222, Q4 DMP2110UW, Q5 DMP2110UW, Q6 MMBT2222, Q7 SiS415DNT, Q8 DMP2110UW, Q9 MMBT2222, U1 Argos_SMD, U10 AH1806-W, U11 LTC3221EDC-3.3, U2 ESP32-S3-WROOM-1, U3 keller_6LHPD, U4 RV-3032-C7, U5 CAM-M8Q, U6 BQ29732, U7 BQ51050BRHL, U8 TPS63001, U9 TPS63900

Commit message: Add second explosive channel and remake layout of J4 and change footprint of Q7
Parts:
- added Q19: MMBT2222, Package_TO_SOT_SMD:SOT-323_SC-70, F.Cu at (135.2, 140.7)
- added Q20: DMP2110UW, Package_TO_SOT_SMD:SOT-323_SC-70, F.Cu at (134.6, 144.4)
- added R56: 100k, Resistor_SMD:R_0402_1005Metric, F.Cu at (134.6, 142.4)
- added R57: 100k, Resistor_SMD:R_0402_1005Metric, F.Cu at (138.3, 140.8)
- added R58: 100k, Resistor_SMD:R_0402_1005Metric, F.Cu at (140.0, 140.3)
- J4: footprint myDevices:PadArray_SMD_1x04_P1.27mm -> myDevices:PadArray_SMD_1x05_P1.27mm; moved to B.Cu
- Q7: value SiS415DNT -> DMP2110UW; footprint Package_SO:Vishay_PowerPAK_1212-8_Single -> Package_TO_SOT_SMD:SOT-323_SC-70
- moved Q7 21.6 mm to (113.9, 110.0)
- moved Q4 7.32 mm to (139.2, 148.1)
- moved R23 7.21 mm to (139.2, 145.8), turned to 0 degrees
- moved R25 3.20 mm to (137.4, 147.3), turned to -90 degrees
- moved R27 2.63 mm to (140.1, 142.7), turned to -90 degrees
- moved Q6 2.42 mm to (137.8, 144.0), turned to 0 degrees
- moved R22 2.28 mm to (136.3, 147.3), turned to 90 degrees
- moved R26 2.24 mm to (138.3, 142.2)
- moved J4 0.81 mm to (136.5, 147.4), turned to 180 degrees
Connections:
- net /EXP_EN renamed /EXP1_EN
- Q7 pad 1: /Batt -> Net-(Q11-C)
- Q7 pad 3: /Batt -> Net-(J6-Pin_2)
- U2 pad 34: unconnected-(U2-IO41-Pad34) -> /EXP2_EN
Routing:
- net /3V3: track 190.4 -> 177.4 mm
- net GND: track 89.7 -> 99.1 mm, vias 119 -> 117
- net /Batt: track 176.4 -> 184.7 mm, vias 35 -> 36
- net /I2C1_SCL: track 22.8 -> 18.1 mm
- net Net-(Q19-C): track 0.00 -> 3.38 mm
- net /I2C1_SDA: track 22.9 -> 19.8 mm
- net /EXP2_EN: track 0.00 -> 2.88 mm
- net Net-(Q4-G): track 6.78 -> 3.91 mm
- net Net-(J4-Pin_5): track 0.00 -> 1.95 mm, vias 0 -> 1
- net Net-(Q19-B): track 0.00 -> 1.92 mm
- net /AS5510_EN: track 4.47 -> 2.85 mm
- net Net-(Q6-B): track 3.43 -> 1.91 mm
- net Net-(J4-Pin_4): track 6.91 -> 7.63 mm, vias 0 -> 1
- net /power/BAT-: vias 18 -> 17
- added copper zone on F.Cu, net Net-(J4-Pin_5)
