File: uterotrack.kicad_sch (KiCad schematic)
At the start: 77 parts, among them J1 RFShield, J2 MicroSD_Card, J3 Argos_Prog, J4 AS5510, J5 Prog, J6 EXP, Q1 DMP2110UW, Q10 MMBT2222, Q11 MMBT2222, Q12 MMBT2222, Q13 MMBT2222, Q2 DMP2110UW, Q3 MMBT2222, Q4 DMP2110UW, Q5 DMP2110UW, Q6 MMBT2222, Q7 SiS415DNT, Q8 DMP2110UW, Q9 MMBT2222, U1 Argos_SMD, U2 ESP32-S3-WROOM-1, U3 keller_6LHPD, U4 RV-3032-C7, U5 CAM-M8Q

Commit message: Add second explosive channel and remake layout of J4 and change footprint of Q7
Parts:
- removed J4: AS5510, myDevices:PadArray_SMD_1x04_P1.27mm, symbol Connector_Generic:Conn_01x04
- removed Q7: SiS415DNT, Package_SO:Vishay_PowerPAK_1212-8_Single, symbol Transistor_FET:SiS415DNT
- added J4: AS5510, myDevices:PadArray_SMD_1x05_P1.27mm, symbol Connector_Generic:Conn_01x05
- added Q19: MMBT2222, Package_TO_SOT_SMD:SOT-323_SC-70, symbol Transistor_BJT:Q_NPN_BEC
- added Q20, Q7: DMP2110UW, Package_TO_SOT_SMD:SOT-323_SC-70, symbol Transistor_FET:Q_PMOS_GSD
- added R56, R57, R58: 100k, Resistor_SMD:R_0402_1005Metric, symbol Device:R
Connections:
- net Batt: now also Q20.2 (S), Q7.2 (S), R56.1
- net GND: now also J4.1 (Pin_1), Q19.2 (E), R58.2
- net I2C1_SCL: now also J4.3 (Pin_3)
- net I2C1_SDA: now also J4.2 (Pin_2)
- net at Q4.3 (D), R22.1, R25.2: now also J4.4 (Pin_4)
- net at Q11.3 (C), R28.2: now also Q7.1 (G)
- net at J6.2 (Pin_2): now also Q7.3 (D)
- net EXP2_EN: now reaches U2.34 (IO41)
- net EXP2_EN: now also R57.1, R58.1
- net EXP_EN renamed EXP1_EN
- new net: Q19.3 (C), Q20.1 (G), R56.2
- new net: J4.5 (Pin_5), Q20.3 (D)
- new net: Q19.1 (B), R57.2
- no-connect marks 29 -> 28
Other:
- moved on the sheet: Q6, R22, R23, R25, R26, R27
